File: flex/flex.kicad_pcb (KiCad board)
At the start: 2 copper layers, 126.5 x 148.9 mm, 83 parts, among them J1 Conn_01x06_Female, J10 Conn_01x02_Female, J11 Conn_01x02_Female, J12 Conn_01x02_Female, J13 Conn_01x02_Female, J14 Conn_01x06_Female, J15 Conn_01x02_Female, J2 Conn_01x07_Female, J3 Conn_01x02_Female, J4 Conn_01x02_Female, J5 Conn_01x02_Female, J6 Conn_01x02_Female, J7 Conn_01x02_Female, J8 Conn_01x02_Female, J9 Conn_01x02_Female, SW1 SW_Push, SW10 SW_Push, SW11 SW_Push, SW12 SW_Push, SW13 SW_Push, SW14 SW_Push, SW15 SW_Push, SW16 SW_Push, SW17 SW_Push, SW18 SW_Push, SW19 SW_Push, SW2 SW_Push, SW20 SW_Push, SW21 SW_Push, SW22 SW_Push, SW23 SW_Push, SW24 SW_Push, SW25 SW_Push, SW26 SW_Push, SW27 SW_Push, SW28 SW_Push, SW29 SW_Push, SW3 SW_Push, SW30 SW_Push, SW31 SW_Push, SW32 SW_Push, SW4 SW_Push, SW5 SW_Push, SW6 SW_Push, SW7 SW_Push, SW8 SW_Push, SW9 SW_Push

Commit message: Add files via upload
Parts:
- added J14: Conn_01x06_Female, Connector_PinSocket_2.54mm:PinSocket_1x06_P2.54mm_Vertical, F.Cu at (57.7, 102.3)
- added J14: Conn_01x06_Female, Connector_PinSocket_2.54mm:PinSocket_1x06_P2.54mm_Vertical, F.Cu at (100.3, 134.3)
- added J2: Conn_01x07_Female, Connector_PinSocket_2.54mm:PinSocket_1x07_P2.54mm_Vertical, F.Cu at (100.9, 119.2)
- added J2: Conn_01x07_Female, Connector_PinSocket_2.54mm:PinSocket_1x07_P2.54mm_Vertical, F.Cu at (57.5, 86.8)
- added J3: Conn_01x02_Female, customs2:SolderWire-0.15sqmm_1x01_D0.5mm_OD1.5mm, F.Cu at (160.4, 51.4)
- added J4: Conn_01x02_Female, customs2:SolderWire-0.15sqmm_1x01_D0.5mm_OD1.5mm, F.Cu at (40.7, 85.4)
- added J4: Conn_01x02_Female, customs2:SolderWire-0.15sqmm_1x01_D0.5mm_OD1.5mm, F.Cu at (160.5, 75.1)
- added J5: Conn_01x02_Female, customs2:SolderWire-0.15sqmm_1x01_D0.5mm_OD1.5mm, F.Cu at (40.6, 108.0)
- added J5: Conn_01x02_Female, customs2:SolderWire-0.15sqmm_1x01_D0.5mm_OD1.5mm, F.Cu at (163.4, 96.4)
- added J6: Conn_01x02_Female, customs2:SolderWire-0.15sqmm_1x01_D0.5mm_OD1.5mm, F.Cu at (163.2, 101.0)
- added J6: Conn_01x02_Female, customs2:SolderWire-0.15sqmm_1x01_D0.5mm_OD1.5mm, F.Cu at (40.6, 112.4)
- added J7: Conn_01x02_Female, customs2:SolderWire-0.15sqmm_1x01_D0.5mm_OD1.5mm, F.Cu at (163.5, 117.7)
- added J7: Conn_01x02_Female, customs2:SolderWire-0.15sqmm_1x01_D0.5mm_OD1.5mm, F.Cu at (53.0, 129.2)
- J1: value Conn_01x06_Female -> Conn_01x08_Female
- moved J8 24.2 mm to (83.8, 138.0)
- moved J14 20.1 mm to (123.9, 100.6)
- moved D1 20.1 mm to (51.1, 81.0)
- moved D10 20.1 mm to (95.3, 90.4)
- moved D11 20.1 mm to (95.3, 113.7)
- moved D13 20.1 mm to (95.5, 159.5)
- moved D15 20.1 mm to (117.4, 88.4)
- moved D18 20.1 mm to (117.4, 157.5)
- moved D20 20.1 mm to (140.5, 91.7)
- moved D21 20.1 mm to (140.5, 114.1)
- moved D22 20.1 mm to (140.7, 137.4)
- moved D4 20.1 mm to (51.1, 149.8)
- moved D6 20.1 mm to (73.4, 103.6)
- moved D8 20.1 mm to (73.4, 149.1)
- moved G*** 20.1 mm to (147.3, 152.8)
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Connections:
- D1 pad 1: col1 -> col0
- D10 pad 1: col3 -> col2
- D11 pad 1: col3 -> col2
- D12 pad 1: col3 -> col2
- D13 pad 1: col3 -> col2
- D14 pad 1: col4 -> col3
- D15 pad 1: col4 -> col3
- D16 pad 1: col4 -> col3
- D17 pad 1: col4 -> col3
- D18 pad 1: col4 -> col3
- D19 pad 1: col5 -> col4
- D2 pad 1: col1 -> col0
- D20 pad 1: col5 -> col4
- D21 pad 1: col5 -> col4
- D22 pad 1: col5 -> col4
- D23 pad 1: col6 -> col5
- D24 pad 1: col6 -> col5
- D25 pad 1: col6 -> col5
- D26 pad 1: col6 -> col5
- D27 pad 1: col1 -> col0
- D28 pad 1: col2 -> col1
- D29 pad 1: col3 -> col2
- D3 pad 1: col1 -> col0
- D30 pad 1: col4 -> col3
- D31 pad 1: col5 -> col4
- D32 pad 1: col6 -> col5
- D4 pad 1: col1 -> col0
- D5 pad 1: col2 -> col1
- D6 pad 1: col2 -> col1
- D7 pad 1: col2 -> col1
- D8 pad 1: col2 -> col1
- D9 pad 1: col3 -> col2
- J1 pad 1: row6 -> row5
- J1 pad 2: col2 -> col1
- J1 pad 3: col3 -> col2
- J1 pad 4: col4 -> col3
- J1 pad 5: col5 -> col4
- J1 pad 6: col6 -> col5
- J10 pad 1: col2 -> col1
- J11 pad 1: col3 -> col2
- J12 pad 1: col4 -> col3
- J13 pad 1: col5 -> col4
- J14 pad 1: col1 -> col0
- J14 pad 2: col2 -> col1
- J14 pad 3: col3 -> col2
- J14 pad 4: col4 -> col3
- J14 pad 5: col5 -> col4
- J14 pad 6: col6 -> col5
- J15 pad 1: col6 -> col5
- J9 pad 1: col1 -> col0
Routing:
- net col0: track 0.00 -> 386.1 mm, vias 0 -> 3
- net col6: track 277.0 -> 0.00 mm, vias 1 -> 0
- net row0: track 916.0 -> 1000.3 mm, vias 2 -> 5
- net row1: track 770.4 -> 845.5 mm, vias 1 -> 5
- net row3: track 347.0 -> 421.7 mm, vias 2 -> 5
- net col5: track 210.8 -> 283.8 mm, vias 0 -> 3
- net col3: track 274.1 -> 205.5 mm, vias 3 -> 2
- net row4: track 463.2 -> 504.8 mm, vias 0 -> 3
- net row2: track 538.4 -> 577.3 mm, vias 3 -> 5
- net col2: track 306.4 -> 272.9 mm, vias 3 -> 6
- net col1: track 329.3 -> 359.5 mm, vias 1 -> 6
- net row5: track 184.0 -> 203.8 mm, vias 2 -> 4
- net row6: track 53.0 -> 64.1 mm, vias 1 -> 2
- net col4: track 210.5 -> 213.6 mm, vias 2 -> 3
Other:
- board size 126.5 x 148.9 mm -> 126.5 x 148.8 mm
- board text added: "C0"
- board text added: "C0R0"
- board text added: "C0R1"
- board text added: "C0R2"
- board text added: "C0R3"
- board text added: "C0R4"
- board text added: "C2R5"
- board text added: "Crystal Keebs"
- board text added: "Dactyl Cut Here"
- board text added: "Dactyl Pinkie columns"
- board text added: "Thumb Cluster"
- board text added: "With modifications by crystalhand v.1"
- board text added: "With modifications by crystalhand v.2"
- board text added: "With modifications made by crystalhand v.2"
- board text removed: "C4R5"
- board text removed: "C6"
- board text removed: "C6R0"
- board text removed: "C6R1"
- board text removed: "C6R2"
- board text removed: "C6R3"
- board text removed: "C6R4"
